Commit message: added camera to xacros

File: catkin_ws/src/my_robot/urdf/my_robot.xacro (robot description, xacro)
@@ -117,4 +117,30 @@
     <dynamics damping="1.0" friction="1.0"/>
   </joint>
--->
+  <link name='camera'>
+    <inertial>
+      <mass value="0.1"/>
+      <origin xyz="0.05 0.05 0.05" rpy="0 0 0"/>
+      <inertia
+         ixx="1e-6" ixy="0" ixz="0" iyy="1e-6" iyz="0" izz="1e-6"
+      />
+    </inertial>
+    <collision name='camera_collision'>
+      <origin xyz="0 0 0" rpy="0 0 0"/>
+      <geometry>
+          <box size="0.05 0.05 0.05"/>
+      </geometry>
+    </collision>
+    <visual name='camera_visual'>
+      <origin xyz="0 0 0" rpy="0 0 0"/>
+      <geometry>
+          <box size="0.05 0.05 0.05"/>
+      </geometry>
+    </visual>
+  </link>
+  <joint type="fixed" name="camera_joint">
+    <origin xyz="0.2 0 0.0" rpy="0 0 0"/>
+    <child link="camera"/>
+    <parent link="chassis"/>
+    <axis xyz="0 1 0" rpy="0 0 0"/>
+  </joint>
 </robot>

Commit message: added lidar

File: catkin_ws/src/my_robot/urdf/my_robot.xacro (robot description, xacro)
@@ -144,3 +144,30 @@
     <axis xyz="0 1 0" rpy="0 0 0"/>
   </joint>
+  <link name='hokuyo'>
+    <inertial>
+      <mass value="1e-5"/>
+      <origin xyz="0 0 0" rpy="0 0 0"/>
+      <inertia
+         ixx="1e-6" ixy="0" ixz="0" iyy="1e-6" iyz="0" izz="1e-6"
+      />
+    </inertial>
+    <collision name='camera_collision'>
+      <origin xyz="0 0 0" rpy="0 0 0"/>
+      <geometry>
+          <box size="0.1 0.1 0.1"/>
+      </geometry>
+    </collision>
+    <visual name='camera_visual'>
+      <origin xyz="0 0 0" rpy="0 0 0"/>
+      <geometry>
+          <mesh filename="package://my_robot/meshes/hokuyo.dae"/>
+      </geometry>
+    </visual>
+  </link>
+  <joint type="fixed" name="hokuyo_joint">
+    <origin xyz="0.15 0 0.1" rpy="0 0 0"/>
+    <child link="hokuyo"/>
+    <parent link="chassis"/>
+    <axis xyz="0 1 0" rpy="0 0 0"/>
+  </joint>
 </robot>

Commit message: robot renders correctly but wont drive
maybe issue with castor friction?

File: catkin_ws/src/my_robot/urdf/my_robot.xacro (robot description, xacro)
@@ -1,10 +1,10 @@
 <?xml version='1.0'?>
 <robot name="my_robot" xmlns:xacro="http://www.ros.org/wiki/xacro">
-  <xacro:include filename="$(find my_robot)/urdf/my_robot.gazebo" />
+  <xacro:include filename="$(find my_robot)/urdf/my_robot.gazebo"/>
   <link name="robot_footprint"></link>
   <joint name="robot_footprint_joint" type="fixed">
-    <origin xyz="0 0 0" rpy="0 0 0" />
+    <origin xyz="0 0 0" rpy="0 0 0"/>
     <parent link="robot_footprint"/>
-    <child link="chassis" />
+    <child link="chassis"/>
   </joint>
   <link name='chassis'>
@@ -13,22 +13,66 @@
       <mass value="15.0"/>
       <origin xyz="0.0 0 0" rpy=" 0 0 0"/>
-      <inertia
-          ixx="0.1" ixy="0" ixz="0"
-          iyy="0.1" iyz="0"
-          izz="0.1"
-      />
-    </inertial>
-    <collision name='collision'>
-      <origin xyz="0 0 0" rpy=" 0 0 0"/>
-      <geometry>
-        <box size=".4 .2 .1"/>
-      </geometry>
-    </collision>
-    <visual name='chassis_visual'>
-      <origin xyz="0 0 0" rpy=" 0 0 0"/>
-      <geometry>
-        <box size=".4 .2 .1"/>
-      </geometry>
-    </visual>
+      <inertia ixx="0.1" ixy="0" ixz="0" iyy="0.1" iyz="0" izz="0.1"/>
+    </inertial>
+    <collision name='chassis_axle_collision'>
+      <origin xyz="0.15 0 0" rpy="0 1.5707 1.5707"/>
+      <geometry>
+        <cylinder length="0.2" radius="0.025"/>
+      </geometry>
+    </collision>
+    <visual name='chassis_axle_visual'>
+      <origin xyz="0.15 0 0" rpy="0 1.5707 1.5707"/>
+      <geometry>
+        <cylinder length="0.2" radius="0.025"/>
+      </geometry>
+      <material name="black">
+        <color rgba="0 0 0 1.0"/>
+      </material>
+    </visual>
+    <visual name='chassis_main_visual'>
+      <origin xyz="-0.05 0 -0.00" rpy=" 0 1.5707 0"/>
+      <geometry>
+          <cylinder length="0.3" radius="0.025"/>
+      </geometry>
+      <material name="dark_purple">
+        <color rgba="0.5 0.05 0.5 1.0"/>
+      </material>
+    </visual>
+    <collision name='chassis_main_collision'>
+      <origin xyz="-0.05 0 -0.00" rpy=" 0 1.5707 0"/>
+      <geometry>
+          <cylinder length="0.3" radius="0.025"/>
+      </geometry>
+    </collision>
+    <visual name='chassis_caster_mount_visual'>
+      <origin xyz="-0.15 0 -0.01" rpy=" 0 0 0"/>
+      <geometry>
+        <box size=".1 .1 .08"/>
+      </geometry>
+      <material name="dark_purple">
+        <color rgba="0.5 0.05 0.5 1.0"/>
+      </material>
+    </visual>
+    <collision name='chassis_caster_mount_collision'>
+      <origin xyz="-0.15 0 -0.01" rpy=" 0 0 0"/>
+      <geometry>
+        <box size=".1 .1 .08"/>
+      </geometry>
+    </collision>
+    <visual name='chassis_lidar_mount_visual'>
+      <origin xyz="0.15 0 0.02" rpy=" 0 0 0"/>
+      <geometry>
+        <box size=".1 .1 .1"/>
+      </geometry>
+        <material name="dark_purple">
+          <color rgba="0.4 0.05 0.4 1.0"/>
+        </material>
+    </visual>
+    <collision name='chassis_lidar_mount_collision'>
+      <origin xyz="0.15 0 0.02" rpy=" 0 0 0"/>
+      <geometry>
+        <box size=".1 .1 .1"/>
+      </geometry>
+    </collision>
     <collision name='back_caster_collision'>
       <origin xyz="-0.15 0 -0.05" rpy=" 0 0 0"/>
@@ -42,16 +86,7 @@
         <sphere radius="0.05"/>
       </geometry>
-    </visual>
-    <collision name='front_caster_collision'>
-      <origin xyz="0.15 0 -0.05" rpy=" 0 0 0"/>
-      <geometry>
-        <sphere radius="0.0499"/>
-      </geometry>
-    </collision>
-    <visual name='front_caster_visual'>
-      <origin xyz="0.15 0 -0.05" rpy=" 0 0 0"/>
-      <geometry>
-        <sphere radius="0.05"/>
-      </geometry>
+      <material name="dark_grey">
+        <color rgba="0.1 0.01 0.01 1.0"/>
+      </material>
     </visual>
   </link>
@@ -60,9 +95,5 @@
       <mass value="5"/>
       <origin xyz="0 0 0" rpy="0 1.5707 1.5707"/>
-      <inertia
-          ixx="0.1" ixy="0" ixz="0"
-          iyy="0.1" iyz="0"
-          izz="0.1"
-      />
+      <inertia ixx="0.1" ixy="0" ixz="0" iyy="0.1" iyz="0" izz="0.1"/>
     </inertial>
     <collision name='left_wheel_collision'>
@@ -77,8 +108,11 @@
         <cylinder length="0.05" radius="0.1"/>
       </geometry>
+      <material name="dark_grey">
+        <color rgba="0.05 0.05 0.05 1.0"/>
+      </material>
     </visual>
   </link>
   <joint type="continuous" name="left_wheel_hinge">
-    <origin xyz="0 0.15 0" rpy="0 0 0"/>
+    <origin xyz="0.15 0.15 0" rpy="0 0 0"/>
     <child link="left_wheel"/>
     <parent link="chassis"/>
@@ -90,10 +124,6 @@
     <inertial>
       <mass value="5"/>
-      <origin xyz="0 0 0" rpy="0 1.5707 1.5707"/>
-      <inertia
-          ixx="0.1" ixy="0" ixz="0"
-          iyy="0.1" iyz="0"
-          izz="0.1"
-      />
+      <origin xyz="0.15 0 0" rpy="0 1.5707 1.5707"/>
+      <inertia ixx="0.1" ixy="0" ixz="0" iyy="0.1" iyz="0" izz="0.1"/>
     </inertial>
     <collision name='right_wheel_collision'>
@@ -108,8 +138,11 @@
         <cylinder length="0.05" radius="0.1"/>
       </geometry>
+      <material name="dark_grey">
+        <color rgba="0.05 0.05 0.05 1.0"/>
+      </material>
     </visual>
   </link>
   <joint type="continuous" name="right_wheel_hinge">
-    <origin xyz="0 -0.15 0" rpy="0 0 0"/>
+    <origin xyz="0.15 -0.15 0" rpy="0 0 0"/>
     <child link="right_wheel"/>
     <parent link="chassis"/>
@@ -122,12 +155,10 @@
       <mass value="0.1"/>
       <origin xyz="0.05 0.05 0.05" rpy="0 0 0"/>
-      <inertia
-         ixx="1e-6" ixy="0" ixz="0" iyy="1e-6" iyz="0" izz="1e-6"
-      />
+      <inertia ixx="1e-6" ixy="0" ixz="0" iyy="1e-6" iyz="0" izz="1e-6"/>
     </inertial>
     <collision name='camera_collision'>
       <origin xyz="0 0 0" rpy="0 0 0"/>
       <geometry>
-          <box size="0.05 0.05 0.05"/>
+        <box size="0.05 0.05 0.05"/>
       </geometry>
     </collision>
@@ -135,5 +166,5 @@
       <origin xyz="0 0 0" rpy="0 0 0"/>
       <geometry>
-          <box size="0.05 0.05 0.05"/>
+        <box size="0.05 0.05 0.05"/>
       </geometry>
     </visual>
@@ -149,12 +180,10 @@
       <mass value="1e-5"/>
       <origin xyz="0 0 0" rpy="0 0 0"/>
-      <inertia
-         ixx="1e-6" ixy="0" ixz="0" iyy="1e-6" iyz="0" izz="1e-6"
-      />
+      <inertia ixx="1e-6" ixy="0" ixz="0" iyy="1e-6" iyz="0" izz="1e-6"/>
     </inertial>
     <collision name='camera_collision'>
       <origin xyz="0 0 0" rpy="0 0 0"/>
       <geometry>
-          <box size="0.1 0.1 0.1"/>
+        <box size="0.1 0.1 0.1"/>
       </geometry>
     </collision>
@@ -162,5 +191,5 @@
       <origin xyz="0 0 0" rpy="0 0 0"/>
       <geometry>
-          <mesh filename="package://my_robot/meshes/hokuyo.dae"/>
+        <mesh filename="package://my_robot/meshes/hokuyo.dae"/>
       </geometry>
     </visual>
